Commit message: fixes after testing

File: src/station/config/srdf/default_setup.srdf.xacro (robot description, xacro)
@@ -10,5 +10,6 @@
   <xacro:include filename="$(find cameras)/srdf/basler.srdf.xacro"/>
   <xacro:include filename="$(find laser_sensors)/srdf/cross_laser.srdf.xacro"/>
-  <xacro:include filename="$(find endtools)/srdf/dispensing_tool.srdf.xacro"/>
+  <xacro:include filename="$(find tools_manager)/srdf/tool_mount.srdf.xacro"/>
+  <xacro:include filename="$(find tools_manager)/srdf/tool_rack.srdf.xacro"/>
   <xacro:macro name="ur_srdf" params="">
     <!--GROUPS - Representation of a set of joints and links. This can be useful for specifying DOF to plan for, defining arms, end effectors, etc-->
@@ -45,20 +46,14 @@
     <disable_collisions link1="ground_plane" link2="base_link" reason="Adjacent" />
     <disable_collisions link1="ground_plane" link2="base_link_inertia" reason="Adjacent" />
-    <disable_collisions link1="tool_mount_link" link2="tool0" reason="Adjacent" />
-    <disable_collisions link1="tool_mount_link" link2="flange" reason="Never" />
-    <disable_collisions link1="tool_mount_link" link2="wrist_1_link" reason="Never" />
-    <disable_collisions link1="tool_mount_link" link2="wrist_2_link" reason="Never" />
-    <disable_collisions link1="tool_mount_link" link2="wrist_3_link" reason="Never" />
     <!-- Disable collisions between the camera and the link it is mounted on -->
-    <xacro:basler_camera_srdf parent="tool_mount_link" name="basler" />
+    <xacro:basler_camera_srdf parent="tool_mount_tcp" name="basler" />
     <xacro:basler_camera_srdf parent="flange" name="basler" />
     <xacro:basler_camera_srdf parent="wrist_3_link" name="basler" />
     <!-- Disable collisions between the laser sensor and the link it is mounted on -->
     <xacro:cross_laser_srdf parent="station" name="captron"/>
-    <!-- Disable collisions between the dispensing tool and the link it is mounted on -->
-    <xacro:dispensing_tool_srdf parent="tool_mount_link" name="dispensing"/>
-    <xacro:dispensing_tool_srdf parent="flange" name="dispensing" />
-    <xacro:dispensing_tool_srdf parent="wrist_3_link" name="dispensing" />
-    <xacro:dispensing_tool_srdf parent="basler_camera_link" name="dispensing" />
+    <!-- Disable collisions between the tool mount and the wrist links it touches -->
+    <xacro:tool_mount_srdf touch_links="wrist_1_link wrist_2_link wrist_3_link"/>
+    <!-- Disable collision between the tool rack and the link it is mounted on -->
+    <xacro:tool_rack_srdf parent="station"/>
   </xacro:macro>
   <xacro:ur_srdf/>

File: src/station/config/urdf/ur/gz_sim.urdf.xacro (robot description, xacro)
@@ -99,6 +99,6 @@
     parent="station"
     simulated="true"
-    rack_origin_xyz="0.35 -0.4 0.9"
-    rack_origin_rpy="0 0 0"
+    rack_origin_xyz="0.3 -0.7 0.9"
+    rack_origin_rpy="0 0 1.5708"
     number_of_slots="2"
     slot_spacing="-0.25"
@@ -127,6 +127,6 @@
     parent="tool0"
     simulated="true"
-    mount_origin_xyz="0.0272 0 0"
-    mount_origin_rpy="0 0 0"
+    mount_origin_xyz="0 0 0.0272"
+    mount_origin_rpy="0 -1.5708 -1.5708"
   />
   <xacro:basler_camera parent="tool_mount_tcp" name="basler" simulated="true" tf_prefix="$(arg tf_prefix)">

File: src/station/config/urdf/ur/real.urdf.xacro (robot description, xacro)
@@ -140,6 +140,6 @@
     parent="tool0"
     simulated="false"
-    mount_origin_xyz="0.0272 0 0"
-    mount_origin_rpy="0 0 0"
+    mount_origin_xyz="0 0 0.0272"
+    mount_origin_rpy="0 -1.5708 -1.5708"
   />
   <xacro:basler_camera parent="tool_mount_tcp" name="basler" simulated="false" tf_prefix="$(arg tf_prefix)">

File: src/tools_manager/urdf/tool_mount.urdf.xacro (robot description, xacro)
@@ -1,4 +1,9 @@
 <?xml version="1.0"?>
 <tool_mount xmlns:xacro="http://wiki.ros.org/xacro">
+  <!--
+    NOTE: Collisions between 'tool_mount_tcp' and its touch links are disabled
+    in the SRDF (see tools_manager/srdf/tool_mount.srdf.xacro), NOT here.
+    disable_collisions is an SRDF-only concept; MoveIt ignores it in the URDF.
+  -->
   <xacro:macro name="tool_mount" params="
     parent:=tool0
@@ -11,5 +16,5 @@
             <origin xyz="0 0 0" rpy="0 0 0"/>
             <geometry>
-                <mesh filename="model://tool_mount/meshes/visual.dae"/>
+                <mesh filename="file://$(find tools_manager)/model/tool_mount/meshes/visual.dae"/>
             </geometry>
         </visual>
@@ -17,5 +22,5 @@
             <origin xyz="0 0 0" rpy="0 0 0"/>
             <geometry>
-                <mesh filename="model://tool_mount/meshes/collision.stl"/>
+                <mesh filename="file://$(find tools_manager)/model/tool_mount/meshes/collision.stl"/>
             </geometry>
         </collision>
@@ -32,5 +37,4 @@
         </inertial>
     </link>
-    <disable_collisions link1="tool_mount_tcp" link2="${parent}" reason="Adjacent" />
     <joint name="tool_mount_tcp_joint" type="fixed">
         <parent link="${parent}"/>
@@ -38,6 +42,22 @@
         <origin xyz="${mount_origin_xyz}" rpy="${mount_origin_rpy}"/>
     </joint>
+    <!--
+        Keep 'tool_mount_tcp' as a real SDF <link> so the tool model's Gazebo
+        DetachableJoint can resolve it via model.LinkByName(). Without
+        preserveFixedJoint the URDF->SDF converter lumps this fixed-joint child
+        into its parent and demotes it to a <frame>, which the plugin cannot
+        find (resulting in "Child Link tool_mount_tcp could not be found").
+    -->
+    <gazebo reference="tool_mount_tcp_joint">
+        <preserveFixedJoint>true</preserveFixedJoint>
+    </gazebo>
     <xacro:if value="${simulated}">
-        <link name="rfid_scanner_link"/>
+        <link name="rfid_scanner_link">
+            <inertial>
+                <origin xyz="0 0 0" rpy="0 0 0"/>
+                <mass value="1e-6"/>
+                <inertia ixx="1e-9" ixy="0" ixz="0" iyy="1e-9" iyz="0" izz="1e-9"/>
+            </inertial>
+        </link>
         <joint name="tool_mount_to_rfid_scanner_joint" type="fixed">
             <parent link="tool_mount_tcp"/>
@@ -45,4 +65,13 @@
             <origin xyz="0.0778 0 -0.033" rpy="0 0 0"/>
         </joint>
+        <!--
+            Keep the RFID frame as a real SDF <link> so the RfidReader plugin can
+            resolve it via model.LinkByName(). Without preserveFixedJoint the URDF->SDF
+            converter lumps this massless fixed-joint child into its parent and turns it
+            into a <frame>, which the plugin cannot find (link resolver returns null).
+        -->
+        <gazebo reference="tool_mount_to_rfid_scanner_joint">
+            <preserveFixedJoint>true</preserveFixedJoint>
+        </gazebo>
         <gazebo>
             <plugin filename="rfid_sim_systems"

File: src/tools_manager/urdf/tool_rack.urdf.xacro (robot description, xacro)
@@ -20,5 +20,11 @@
     rfid_scanner_origin_rpy:='0 0 0'
     ">
-    <link name="slot${index}_attached_link"/>
+    <link name="slot${index}_attached_link">
+        <inertial>
+            <origin xyz="0 0 0" rpy="0 0 0"/>
+            <mass value="1e-6"/>
+            <inertia ixx="1e-9" ixy="0" ixz="0" iyy="1e-9" iyz="0" izz="1e-9"/>
+        </inertial>
+    </link>
     <joint name="slot${index}_attached_joint" type="fixed">
         <parent link="${parent}"/>
@@ -26,4 +32,16 @@
         <origin xyz="${tool_attached_origin_xyz.split()[0]} ${float(tool_attached_origin_xyz.split()[1]) + float(y_offset)} ${tool_attached_origin_xyz.split()[2]}" rpy="${tool_attached_origin_rpy}"/>
     </joint>
+    <!--
+        Keep 'slot${index}_attached_link' as a real SDF <link> so the tool
+        model's Gazebo DetachableJoint can resolve it via model.LinkByName().
+        Without preserveFixedJoint the URDF->SDF converter lumps this
+        fixed-joint child into its parent and demotes it to a <frame>, which
+        the plugin cannot find (resulting in "Child Link slot${index}_attached_link
+        could not be found"). A tiny inertial block is required too: SDFormat
+        ignores preserveFixedJoint on a massless link and lumps it regardless.
+    -->
+    <gazebo reference="slot${index}_attached_joint">
+        <preserveFixedJoint>true</preserveFixedJoint>
+    </gazebo>
     <link name="slot${index}_lifted_link"/>
     <joint name="slot${index}_lifted_joint" type="fixed">
@@ -39,5 +57,11 @@
     </joint>
     <xacro:if value="${simulated}">
-        <link name="slot${index}_rfid_scanner_link"/>
+        <link name="slot${index}_rfid_scanner_link">
+            <inertial>
+                <origin xyz="0 0 0" rpy="0 0 0"/>
+                <mass value="1e-6"/>
+                <inertia ixx="1e-9" ixy="0" ixz="0" iyy="1e-9" iyz="0" izz="1e-9"/>
+            </inertial>
+        </link>
         <joint name="slot${index}_to_rfid_scanner_joint" type="fixed">
             <parent link="slot${index}_attached_link"/>
@@ -45,4 +69,13 @@
             <origin xyz="${rfid_scanner_origin_xyz.split()[0]} ${float(rfid_scanner_origin_xyz.split()[1]) + float(y_offset)} ${rfid_scanner_origin_xyz.split()[2]}" rpy="${rfid_scanner_origin_rpy}"/>
         </joint>
+        <!--
+            Keep the RFID frame as a real SDF <link> so the RfidReader plugin can
+            resolve it via model.LinkByName(). Without preserveFixedJoint the URDF->SDF
+            converter lumps this massless fixed-joint child into its parent and turns it
+            into a <frame>, which the plugin cannot find (link resolver returns null).
+        -->
+        <gazebo reference="slot${index}_to_rfid_scanner_joint">
+            <preserveFixedJoint>true</preserveFixedJoint>
+        </gazebo>
         <gazebo>
             <plugin filename="rfid_sim_systems"
@@ -61,13 +94,16 @@
     "Loop" over slots. Xacro has no native for-loop, so recursion is used:
     the macro instantiates one slot then calls itself with index+1 until
-    index == count. Each slot is offset along X by `spacing`.
+    index > count. Slot indices are 1-based (slot1, slot2, ...) to match the
+    1-based indices used in the tools_manager config and SlotInfo/ToolInfo
+    messages. Each slot is offset along X by `spacing`, with the first slot
+    (index 1) at zero offset.
   -->
-  <xacro:macro name="tool_slots" params="parent simulated count spacing:=0.15 index:=0">
-    <xacro:if value="${index &lt; count}">
+  <xacro:macro name="tool_slots" params="parent simulated count spacing:=0.15 index:=1">
+    <xacro:if value="${index &lt;= count}">
         <xacro:tool_slot
             simulated="${simulated}"
             index="${index}"
             parent="${parent}"
-            y_offset="${index * spacing}"/>
+            y_offset="${(index - 1) * spacing}"/>
         <xacro:tool_slots
             simulated="${simulated}"
@@ -91,5 +127,5 @@
             <origin xyz="0 0 0" rpy="0 0 0"/>
             <geometry>
-                <mesh filename="model://tool_rack/meshes/visual.dae"/>
+                <mesh filename="file://$(find tools_manager)/model/tool_rack/meshes/visual.dae"/>
             </geometry>
         </visual>
@@ -97,5 +133,5 @@
             <origin xyz="0 0 0" rpy="0 0 0"/>
             <geometry>
-                <mesh filename="model://tool_rack/meshes/collision.stl"/>
+                <mesh filename="file://$(find tools_manager)/model/tool_rack/meshes/collision.stl"/>
             </geometry>
         </collision>
@@ -105,5 +141,9 @@
         </inertial>
     </link>
-    <disable_collisions link1="tool_rack_link" link2="${parent}" reason="Adjacent" />
+    <!--
+      NOTE: Collision between 'tool_rack_link' and its parent is disabled in the
+      SRDF (see tools_manager/srdf/tool_rack.srdf.xacro), NOT here.
+      disable_collisions is an SRDF-only concept; MoveIt ignores it in the URDF.
+    -->
     <joint name="tool_rack_joint" type="fixed">
         <parent link="${parent}"/>
