Commit message: fixes after testing

File: src/tools_manager/urdf/tool_mount.urdf.xacro (robot description, xacro)
@@ -78,5 +78,5 @@
                     name="autofactory::rfid::RfidReader">
                 <link>rfid_scanner_link</link>
-                <range>0.02</range>
+                <range>0.1</range>
                 <update_rate>10</update_rate>
                 <detected_topic>/tool_mount_rfid_scanner/detected</detected_topic>

File: src/tools_manager/urdf/tool_rack.urdf.xacro (robot description, xacro)
@@ -17,5 +17,5 @@
     tool_slide_in_origin_xyz:='0.0656 -0.1025 0.287'
     tool_slide_in_origin_rpy:='0 0 0'
-    rfid_scanner_origin_xyz:='-0.02 -0.1025 0.23'
+    rfid_scanner_origin_xyz:='-0.05 0.0 -0.06'
     rfid_scanner_origin_rpy:='0 0 0'
     ">
@@ -67,5 +67,5 @@
             <parent link="slot${index}_attached_link"/>
             <child link="slot${index}_rfid_scanner_link"/>
-            <origin xyz="${rfid_scanner_origin_xyz.split()[0]} ${float(rfid_scanner_origin_xyz.split()[1]) + float(y_offset)} ${rfid_scanner_origin_xyz.split()[2]}" rpy="${rfid_scanner_origin_rpy}"/>
+            <origin xyz="${rfid_scanner_origin_xyz}" rpy="${rfid_scanner_origin_rpy}"/>
         </joint>
         <!--
@@ -82,5 +82,5 @@
                     name="autofactory::rfid::RfidReader">
                 <link>slot${index}_rfid_scanner_link</link>
-                <range>0.1</range>
+                <range>0.15</range>
                 <update_rate>10</update_rate>
                 <detected_topic>/slot${index}_rfid_scanner/detected</detected_topic>
