Commit message: impelement tools_manager node

File: src/endtools/model/dispensing_tool/model.sdf.xacro (robot description, xacro)
@@ -7,4 +7,5 @@
         tool_mount_link:=tool_mount_tcp
         tool_rack_link:=slot1_attached_link
+        tag_data:=6162633132330020202020202020202044495350454E53494E470020202020204B5243313233002020202020202020205231410020202020202020202020202053584E3132330020202020202020202052314100202020202020202020202020
       ">
     <model name="${model_name}">
@@ -68,4 +69,9 @@
           <output_topic>/${tool_rack_link}/${model_name}/state</output_topic>
       </plugin>
+      <plugin filename="rfid_sim_systems"
+              name="autofactory::rfid::RfidTag">
+        <id>${model_name}</id>
+        <data encoding="hex">${tag_data}</data>
+      </plugin>
     </model>
   </xacro:macro>

File: src/tools_manager/urdf/tool_mount.urdf.xacro (robot description, xacro)
@@ -3,4 +3,5 @@
   <xacro:macro name="tool_mount" params="
     parent:=tool0
+    simulated:=true
     mount_origin_xyz:='0 0 0'
     mount_origin_rpy:='0 0 0'
@@ -41,4 +42,23 @@
         <origin xyz="${tcp_origin_xyz}" rpy="${tcp_origin_rpy}"/>
     </joint>
+    <xacro:if value="${simulated}">
+        <link name="rfid_scanner_link"/>
+        <joint name="tool_mount_to_rfid_scanner_joint" type="fixed">
+            <parent link="tool_mount_link"/>
+            <child link="rfid_scanner_link"/>
+            <origin xyz="0 0 0" rpy="0 0 0"/>
+        </joint>
+        <gazebo>
+            <plugin filename="rfid_sim_systems"
+                    name="autofactory::rfid::RfidReader">
+                <link>rfid_scanner_link</link>
+                <range>0.1</range>
+                <update_rate>10</update_rate>
+                <detected_topic>/tool_mount_rfid_scanner/detected</detected_topic>
+                <content_topic>/tool_mount_rfid_scanner/tag_data</content_topic>
+                <reader_id>tool_mount_reader</reader_id>
+            </plugin>
+        </gazebo>
+    </xacro:if>
   </xacro:macro>
 </tool_mount>

File: src/tools_manager/urdf/tool_rack.urdf.xacro (robot description, xacro)
@@ -7,4 +7,5 @@
   -->
   <xacro:macro name="tool_slot" params="
+    simulated:=true
     index:='2'
     parent:='tool_rack_link'
@@ -35,4 +36,23 @@
         <origin xyz="${float(tool_slide_in_origin_xyz.split()[0]) + float(x_offset)} ${tool_slide_in_origin_xyz.split()[1]} ${tool_slide_in_origin_xyz.split()[2]}" rpy="${tool_slide_in_origin_rpy}"/>
     </joint>
+    <xacro:if value="${simulated}">
+        <link name="slot${index}_rfid_scanner_link"/>
+        <joint name="slot${index}_to_rfid_scanner_joint" type="fixed">
+            <parent link="slot${index}_attached_link"/>
+            <child link="slot${index}_rfid_scanner_link"/>
+            <origin xyz="0 0 0" rpy="0 0 0"/>
+        </joint>
+        <gazebo>
+            <plugin filename="rfid_sim_systems"
+                    name="autofactory::rfid::RfidReader">
+                <link>slot${index}_rfid_scanner_link</link>
+                <range>0.1</range>
+                <update_rate>10</update_rate>
+                <detected_topic>/slot${index}_rfid_scanner/detected</detected_topic>
+                <content_topic>/slot${index}_rfid_scanner/tag_data</content_topic>
+                <reader_id>slot${index}_rfid_scanner</reader_id>
+            </plugin>
+        </gazebo>
+    </xacro:if>
   </xacro:macro>
   <!--
@@ -41,11 +61,13 @@
     index == count. Each slot is offset along X by `spacing`.
   -->
-  <xacro:macro name="tool_slots" params="parent count spacing:=0.15 index:=0">
+  <xacro:macro name="tool_slots" params="parent simulated count spacing:=0.15 index:=0">
     <xacro:if value="${index &lt; count}">
         <xacro:tool_slot
+            simulated="${simulated}"
             index="${index}"
             parent="${parent}"
             x_offset="${index * spacing}"/>
         <xacro:tool_slots
+            simulated="${simulated}"
             parent="${parent}"
             count="${count}"
@@ -56,4 +78,5 @@
   <xacro:macro name="tool_rack" params="
     parent:=station
+    simulated:=true
     rack_origin_xyz:='0 0 0'
     rack_origin_rpy:='0 0 0'
@@ -90,7 +113,5 @@
     </joint>
     <!-- Instantiate N slots as children of the rack body -->
-    <xacro:tool_slots parent="tool_rack_link" count="${number_of_slots}" spacing="${slot_spacing}"/>
+    <xacro:tool_slots parent="tool_rack_link" simulated="${simulated}" count="${number_of_slots}" spacing="${slot_spacing}"/>
   </xacro:macro>
-  <link name="station"/>
-  <xacro:tool_rack parent="station"/>
 </tool_rack>

Commit message: fixes

File: src/endtools/model/dispensing_tool/model.sdf.xacro (robot description, xacro)
@@ -80,4 +80,5 @@
   <xacro:arg name="tool_mount_link"             default="tool_mount_tcp"/>
   <xacro:arg name="tool_rack_link"              default="slot1_attached_joint"/>
+  <xacro:arg name="tag_data"                    default="6162633132330020202020202020202044495350454E53494E470020202020204B5243313233002020202020202020205231410020202020202020202020202053584E3132330020202020202020202052314100202020202020202020202020"/>
   <!-- Instantiate the macro so `xacro dispensing_tool.sdf.xacro` emits a complete model.
        Each macro parameter is fed from its matching $(arg ...) so values passed
@@ -89,4 +90,5 @@
       tool_mount_link="$(arg tool_mount_link)"
       tool_rack_link="$(arg tool_rack_link)"
+      tag_data="$(arg tag_data)"
   />
 </sdf>

File: src/station/config/urdf/ur/gz_sim.urdf.xacro (robot description, xacro)
@@ -9,5 +9,6 @@
   <xacro:include filename="$(find cameras)/urdf/basler.urdf.xacro"/>
   <xacro:include filename="$(find laser_sensors)/urdf/cross_laser.urdf.xacro"/>
-  <xacro:include filename="$(find endtools)/urdf/dispensing_tool.urdf.xacro"/>
+  <xacro:include filename="$(find tools_manager)/urdf/tool_mount.urdf.xacro"/>
+  <xacro:include filename="$(find tools_manager)/urdf/tool_rack.urdf.xacro"/>
   <!-- ros2_control macro (merged from ur_gz.ros2_control.xacro) -->
   <xacro:macro name="ur_ros2_control" params="
@@ -94,4 +95,11 @@
     <child link="station"/>
   </joint>
+  <!-- tool rack attached to station -->
+  <xacro:tool_rack parent="station" simulated="true">
+    <rack_origin_xyz>0 0 0</rack_origin_xyz>
+    <rack_origin_rpy>0 0 0</rack_origin_rpy>
+    <number_of_slots>2</number_of_slots>
+    <slot_spacing>0.15</slot_spacing>
+  </xacro:tool_rack>
   <xacro:cross_laser parent="station" name="captron" simulated="true" tf_prefix="$(arg tf_prefix)">
     <origin xyz="0.35 0.45 0.95" rpy="0 0 3.14"/>
@@ -114,33 +122,13 @@
   </xacro:ur_robot>
   <!-- tool mount attached to tool0 -->
-  <link name="tool_mount_link">
-    <visual>
-      <origin xyz="0 0 0" rpy="0 0 0"/>
-      <geometry>
-        <mesh filename="file://$(find station)/config/model/tool_mount/meshes/tool_mount_visual.dae"/>
-      </geometry>
-    </visual>
-    <collision>
-      <origin xyz="0 0 0" rpy="0 0 0"/>
-      <geometry>
-        <mesh filename="file://$(find station)/config/model/tool_mount/meshes/tool_mount_collision.stl"/>
-      </geometry>
-    </collision>
-    <inertial>
-      <mass value="0.5"/>
-      <inertia ixx="0.001" ixy="0" ixz="0" iyy="0.001" iyz="0" izz="0.001"/>
-    </inertial>
-  </link>
-  <joint name="tool_mount_joint" type="fixed">
-    <parent link="$(arg tf_prefix)tool0"/>
-    <child link="tool_mount_link"/>
-    <origin xyz="0 0 0" rpy="-1.57 -1.57 0"/>
-  </joint>
+  <xacro:tool_mount parent="tool0" simulated="true">
+    <mount_origin_xyz>0 0 0</mount_origin_xyz>
+    <mount_origin_rpy>0 0 0</mount_origin_rpy>
+    <tcp_origin_xyz>0 0 0.1</tcp_origin_xyz>
+    <tcp_origin_rpy>0 0 0</tcp_origin_rpy>
+  </xacro:tool_mount>
   <xacro:basler_camera parent="tool_mount_link" name="basler" simulated="true" tf_prefix="$(arg tf_prefix)">
     <origin xyz="-0.03 0.025 -0.057" rpy="1.57 0 1.57"/>
   </xacro:basler_camera>
-  <xacro:dispensing parent="tool_mount_link" name="dispensing" simulated="true" tf_prefix="$(arg tf_prefix)">
-    <origin xyz="0.0475 0 0" rpy="0 0 0"/>
-  </xacro:dispensing>
   <!-- conveyor belt fixed to world frame -->
   <link name="conveyor">

File: src/station/config/urdf/ur/real.urdf.xacro (robot description, xacro)
@@ -10,5 +10,6 @@
   <xacro:include filename="$(find cameras)/urdf/basler.urdf.xacro"/>
   <xacro:include filename="$(find laser_sensors)/urdf/cross_laser.urdf.xacro"/>
-  <xacro:include filename="$(find endtools)/urdf/dispensing_tool.urdf.xacro"/>
+  <xacro:include filename="$(find tools_manager)/urdf/tool_mount.urdf.xacro"/>
+  <xacro:include filename="$(find tools_manager)/urdf/tool_rack.urdf.xacro"/>
   <!-- possible 'ur_type' values: ur3, ur5, ur10, ur3e, ur5e, ur7e, ur10e, ur12e, ur16e, ur8long, ur15, ur18, ur20, ur30 -->
   <!-- the default value should raise an error in case this was called without defining the type -->
@@ -107,4 +108,11 @@
     <child link="station"/>
   </joint>
+  <!-- tool rack attached to station -->
+  <xacro:tool_rack parent="station" simulated="false">
+    <rack_origin_xyz>0 0 0</rack_origin_xyz>
+    <rack_origin_rpy>0 0 0</rack_origin_rpy>
+    <number_of_slots>2</number_of_slots>
+    <slot_spacing>0.15</slot_spacing>
+  </xacro:tool_rack>
   <xacro:cross_laser parent="station" name="captron" simulated="true" tf_prefix="$(arg tf_prefix)">
     <origin xyz="0.35 0.45 0.95" rpy="0 0 3.14"/>
@@ -127,27 +135,10 @@
   </xacro:ur_robot>
   <!-- tool mount attached to tool0 -->
-  <link name="tool_mount_link">
-    <visual>
-      <origin xyz="0 0 0" rpy="0 0 0"/>
-      <geometry>
-        <mesh filename="file://$(find station)/config/model/tool_mount/meshes/tool_mount_visual.dae"/>
-      </geometry>
-    </visual>
-    <collision>
-      <origin xyz="0 0 0" rpy="0 0 0"/>
-      <geometry>
-        <mesh filename="file://$(find station)/config/model/tool_mount/meshes/tool_mount_collision.stl"/>
-      </geometry>
-    </collision>
-    <inertial>
-      <mass value="0.5"/>
-      <inertia ixx="0.001" ixy="0" ixz="0" iyy="0.001" iyz="0" izz="0.001"/>
-    </inertial>
-  </link>
-  <joint name="tool_mount_joint" type="fixed">
-    <parent link="$(arg tf_prefix)tool0"/>
-    <child link="tool_mount_link"/>
-    <origin xyz="0 0 0" rpy="-1.57 -1.57 0"/>
-  </joint>
+  <xacro:tool_mount parent="tool0" simulated="true">
+    <mount_origin_xyz>0 0 0</mount_origin_xyz>
+    <mount_origin_rpy>0 0 0</mount_origin_rpy>
+    <tcp_origin_xyz>0 0 0.1</tcp_origin_xyz>
+    <tcp_origin_rpy>0 0 0</tcp_origin_rpy>
+  </xacro:tool_mount>
   <xacro:basler_camera parent="tool_mount_link" name="basler" simulated="false" tf_prefix="$(arg tf_prefix)">
     <origin xyz="-0.03 0.025 -0.057" rpy="1.57 0 1.57"/>

File: src/tools_manager/urdf/tool_mount.urdf.xacro (robot description, xacro)
@@ -31,4 +31,5 @@
         </inertial>
     </link>
+    <disable_collisions link1="tool_mount_link" link2="${parent}" reason="Adjacent" />
     <joint name="tool_mount_joint" type="fixed">
         <parent link="${parent}"/>

File: src/tools_manager/urdf/tool_rack.urdf.xacro (robot description, xacro)
@@ -107,4 +107,5 @@
         </inertial>
     </link>
+    <disable_collisions link1="tool_rack_link" link2="${parent}" reason="Adjacent" />
     <joint name="tool_rack_joint" type="fixed">
         <parent link="${parent}"/>

Commit message: move tool_mount rfid scanner to another location

File: src/endtools/model/dispensing_tool/model.sdf.xacro (robot description, xacro)
@@ -47,5 +47,5 @@
           <parent>dispensing_tool_origin</parent>
           <child>rfid_tag_link</child>
-          <pose>0.0506 0 -0.033 0 0 0</pose>
+          <pose>-0.0506 0 -0.033 0 0 0</pose>
       </joint>
       <link name="tool_tcp_uncalibrated"/>

File: src/tools_manager/urdf/tool_mount.urdf.xacro (robot description, xacro)
@@ -66,5 +66,5 @@
             <parent link="tool_mount_tcp"/>
             <child link="rfid_scanner_link"/>
-            <origin xyz="0.0778 0 -0.033" rpy="0 0 0"/>
+            <origin xyz="0 0 -0.033" rpy="0 0 0"/>
         </joint>
         <!--
@@ -81,5 +81,5 @@
                     name="autofactory::rfid::RfidReader">
                 <link>rfid_scanner_link</link>
-                <range>0.1</range>
+                <range>0.05</range>
                 <update_rate>10</update_rate>
                 <detected_topic>/tool_mount_rfid_scanner/detected</detected_topic>

File: src/tools_manager/urdf/tool_rack.urdf.xacro (robot description, xacro)
@@ -17,5 +17,5 @@
     tool_slide_in_origin_xyz:='0.0656 -0.1025 0.287'
     tool_slide_in_origin_rpy:='0 0 0'
-    rfid_scanner_origin_xyz:='-0.05 0.0 -0.06'
+    rfid_scanner_origin_xyz:='-0.05 0.0 -0.03'
     rfid_scanner_origin_rpy:='0 0 0'
     ">
@@ -82,5 +82,5 @@
                     name="autofactory::rfid::RfidReader">
                 <link>slot${index}_rfid_scanner_link</link>
-                <range>0.15</range>
+                <range>0.08</range>
                 <update_rate>10</update_rate>
                 <detected_topic>/slot${index}_rfid_scanner/detected</detected_topic>

Commit message: fix bug in endtool unmounting; fix naming for gz bridge nodes

File: src/endtools/model/dispensing_tool/model.sdf.xacro (robot description, xacro)
@@ -7,6 +7,4 @@
         tool_mount_link:=tool_mount_tcp
         tool_rack_link:=slot1_attached_link
-        tcp_origin_xyz:='0.1043 0 -0.267'
-        tcp_origin_rpy:='0 0 0'
         tag_data:=6162633132330020202020202020202044495350454E53494E470020202020204B5243313233002020202020202020205231410020202020202020202020202053584E3132330020202020202020202052314100202020202020202020202020
       ">
@@ -48,10 +46,4 @@
           <child>rfid_tag_link</child>
           <pose>-0.0506 0 -0.033 0 0 0</pose>
-      </joint>
-      <link name="tool_tcp_uncalibrated"/>
-      <joint name="tool_tcp_uncalibrated_joint" type="fixed">
-          <parent>dispensing_tool_origin</parent>
-          <child>tool_tcp_uncalibrated</child>
-          <pose>${tcp_origin_xyz} ${tcp_origin_rpy}</pose>
       </joint>
       <!--

File: src/laser_sensors/urdf/cross_laser.urdf.xacro (robot description, xacro)
@@ -58,4 +58,8 @@
       range <= window_size. The node's 'detection_distance' parameter (default
       0.04 m) decides the interruption threshold.
+      TODO: currently the laser beams are infinetly thin, but real laser has finite thickness
+            of about 1mm; we should model this by having multiple parallel rays that create
+            a cylinderical detection volume, and then the node should report the minimum range if
+            any of the rays are interrupted.
     -->
     <xacro:if value="${simulated}">
