Commit message: update models; add default velocity

File: src/cameras/urdf/basler.urdf.xacro (robot description, xacro)
@@ -75,4 +75,5 @@
       </xacro:unless>
     </link>
+    <disable_collisions link1="${parent}" link2="${name}_camera_link" reason="Adjacent" />
     <joint name="${name}_camera_joint" type="fixed">
       <parent link="${tf_prefix}${parent}"/>
@@ -80,15 +81,20 @@
       <xacro:insert_block name="origin"/>
     </joint>
+    <link name="camera_tcp_uncalibrated"/>
+    <joint name="camera_tcp_uncalibrated_joint" type="fixed">
+        <parent link="${name}_camera_link"/>
+        <child link="camera_tcp_uncalibrated"/>
+        <xacro:if value="${camera_model == 'basler'}">
+            <origin xyz="0.0188 0.0395 -0.0695" rpy="0 0 0"/>
+        </xacro:if>
+        <xacro:unless value="${is_known_model}">
+            <origin xyz="0 0 0" rpy="0 0 0"/>
+        </xacro:unless>
+    </joint>
     <!-- Gazebo plugin for camera sensor: https://sdformat.org/spec/1.12/sensor/#sensor_camera -->
     <xacro:if value="${simulated}">
-          <gazebo reference="${name}_camera_link">
+          <gazebo reference="camera_tcp_uncalibrated">
               <sensor name="${name}_camera_sensor" type="camera">
-                  <xacro:if value="${camera_model == 'basler'}">
-                      <pose>0.0700233 -0.127701 -0.0225334 0 0 -1.57</pose>
-                  </xacro:if>
-                  <!-- Fallback sensor pose for unknown camera models -->
-                  <xacro:unless value="${is_known_model}">
-                      <pose>0 0 0 0 0 0</pose>
-                  </xacro:unless>
+                <pose>0 0 0 0 0 0</pose>
               <always_on>true</always_on>
               <update_rate>${update_rate}</update_rate>

File: src/endtools/model/dispensing_tool/model.sdf.xacro (robot description, xacro)
@@ -7,4 +7,6 @@
         tool_mount_link:=tool_mount_tcp
         tool_rack_link:=slot1_attached_link
+        tcp_origin_xyz:='0.1043 0 -0.267'
+        tcp_origin_rpy:='0 0 0'
         tag_data:=6162633132330020202020202020202044495350454E53494E470020202020204B5243313233002020202020202020205231410020202020202020202020202053584E3132330020202020202020202052314100202020202020202020202020
       ">
@@ -12,13 +14,12 @@
       <link name="dispensing_tool_origin">
         <inertial>
-          <mass> 0.5094651951956418 </mass>
-          <pose> -4.6297522176e-05 -2.7501563919e-02 -2.8689966722e-06 0 0 0 </pose>
+          <mass> 7.063783650845496  </mass>
           <inertia>
-            <ixx>  1.8444458772e-04 </ixx>
-            <ixy> -1.8714769888e-07 </ixy>
-            <ixz>  2.5644282048e-08 </ixz>
-            <iyy>  1.8051069194e-04 </iyy>
-            <iyz>  4.2089057146e-08 </iyz>
-            <izz>  2.0096567452e-04 </izz>
+            <ixx>  0.00011207748967739463 </ixx>
+            <ixy> 1.032237834897387e-07 </ixy>
+            <ixz>  2.690965380322996e-05 </ixz>
+            <iyy>  0.0001003825439622742 </iyy>
+            <iyz>  -2.3925238308720508e-08 </iyz>
+            <izz>  3.538789883197751e-05 </izz>
           </inertia>
         </inertial>
@@ -42,4 +43,16 @@
         </visual>
       </link>
+      <link name="rfid_tag_link"/>
+      <joint name="rfid_tag_link_joint" type="fixed">
+          <parent>dispensing_tool_origin</parent>
+          <child>rfid_tag_link</child>
+          <pose>0.0506 0 -0.033 0 0 0</pose>
+      </joint>
+      <link name="tool_tcp_uncalibrated"/>
+      <joint name="tool_tcp_uncalibrated_joint" type="fixed">
+          <parent>dispensing_tool_origin</parent>
+          <child>tool_tcp_uncalibrated</child>
+          <pose>${tcp_origin_xyz} ${tcp_origin_rpy}</pose>
+      </joint>
       <!--
       IMPORTANT (gz-sim 8.11.0): this plugin STARTS ATTACHED. Its
@@ -72,4 +85,5 @@
               name="autofactory::rfid::RfidTag">
         <id>${model_name}</id>
+        <link>rfid_tag_link</link>
         <data encoding="hex">${tag_data}</data>
       </plugin>
@@ -79,5 +93,5 @@
   <xacro:arg name="station_model_name"          default="station"/>
   <xacro:arg name="tool_mount_link"             default="tool_mount_tcp"/>
-  <xacro:arg name="tool_rack_link"              default="slot1_attached_joint"/>
+  <xacro:arg name="tool_rack_link"              default="slot1_attached_link"/>
   <xacro:arg name="tag_data"                    default="6162633132330020202020202020202044495350454E53494E470020202020204B5243313233002020202020202020205231410020202020202020202020202053584E3132330020202020202020202052314100202020202020202020202020"/>
   <!-- Instantiate the macro so `xacro dispensing_tool.sdf.xacro` emits a complete model.

File: src/station/config/urdf/ur/gz_sim.urdf.xacro (robot description, xacro)
@@ -96,10 +96,12 @@
   </joint>
   <!-- tool rack attached to station -->
-  <xacro:tool_rack parent="station" simulated="true">
-    <rack_origin_xyz>0 0 0</rack_origin_xyz>
-    <rack_origin_rpy>0 0 0</rack_origin_rpy>
-    <number_of_slots>2</number_of_slots>
-    <slot_spacing>0.15</slot_spacing>
-  </xacro:tool_rack>
+  <xacro:tool_rack
+    parent="station"
+    simulated="true"
+    rack_origin_xyz="0.35 -0.4 0.9"
+    rack_origin_rpy="0 0 0"
+    number_of_slots="2"
+    slot_spacing="-0.25"
+  />
   <xacro:cross_laser parent="station" name="captron" simulated="true" tf_prefix="$(arg tf_prefix)">
     <origin xyz="0.35 0.45 0.95" rpy="0 0 3.14"/>
@@ -122,12 +124,12 @@
   </xacro:ur_robot>
   <!-- tool mount attached to tool0 -->
-  <xacro:tool_mount parent="tool0" simulated="true">
-    <mount_origin_xyz>0 0 0</mount_origin_xyz>
-    <mount_origin_rpy>0 0 0</mount_origin_rpy>
-    <tcp_origin_xyz>0 0 0.1</tcp_origin_xyz>
-    <tcp_origin_rpy>0 0 0</tcp_origin_rpy>
-  </xacro:tool_mount>
-  <xacro:basler_camera parent="tool_mount_link" name="basler" simulated="true" tf_prefix="$(arg tf_prefix)">
-    <origin xyz="-0.03 0.025 -0.057" rpy="1.57 0 1.57"/>
+  <xacro:tool_mount
+    parent="tool0"
+    simulated="true"
+    mount_origin_xyz="0.0272 0 0"
+    mount_origin_rpy="0 0 0"
+  />
+  <xacro:basler_camera parent="tool_mount_tcp" name="basler" simulated="true" tf_prefix="$(arg tf_prefix)">
+    <origin xyz="-0.110 0.02 -0.0575" rpy="0.0 0 0.0"/>
   </xacro:basler_camera>
   <!-- conveyor belt fixed to world frame -->

File: src/station/config/urdf/ur/real.urdf.xacro (robot description, xacro)
@@ -109,10 +109,12 @@
   </joint>
   <!-- tool rack attached to station -->
-  <xacro:tool_rack parent="station" simulated="false">
-    <rack_origin_xyz>0 0 0</rack_origin_xyz>
-    <rack_origin_rpy>0 0 0</rack_origin_rpy>
-    <number_of_slots>2</number_of_slots>
-    <slot_spacing>0.15</slot_spacing>
-  </xacro:tool_rack>
+  <xacro:tool_rack
+    parent="station"
+    simulated="false"
+    rack_origin_xyz="0.35 -0.4 0.9"
+    rack_origin_rpy="0 0 0"
+    number_of_slots="2"
+    slot_spacing="-0.25"
+  />
   <xacro:cross_laser parent="station" name="captron" simulated="true" tf_prefix="$(arg tf_prefix)">
     <origin xyz="0.35 0.45 0.95" rpy="0 0 3.14"/>
@@ -135,16 +137,13 @@
   </xacro:ur_robot>
   <!-- tool mount attached to tool0 -->
-  <xacro:tool_mount parent="tool0" simulated="true">
-    <mount_origin_xyz>0 0 0</mount_origin_xyz>
-    <mount_origin_rpy>0 0 0</mount_origin_rpy>
-    <tcp_origin_xyz>0 0 0.1</tcp_origin_xyz>
-    <tcp_origin_rpy>0 0 0</tcp_origin_rpy>
-  </xacro:tool_mount>
-  <xacro:basler_camera parent="tool_mount_link" name="basler" simulated="false" tf_prefix="$(arg tf_prefix)">
-    <origin xyz="-0.03 0.025 -0.057" rpy="1.57 0 1.57"/>
+  <xacro:tool_mount
+    parent="tool0"
+    simulated="false"
+    mount_origin_xyz="0.0272 0 0"
+    mount_origin_rpy="0 0 0"
+  />
+  <xacro:basler_camera parent="tool_mount_tcp" name="basler" simulated="false" tf_prefix="$(arg tf_prefix)">
+    <origin xyz="-0.110 0.02 -0.0575" rpy="0.0 0 0.0"/>
   </xacro:basler_camera>
-  <xacro:dispensing parent="tool_mount_link" name="dispensing" simulated="false" tf_prefix="$(arg tf_prefix)">
-    <origin xyz="0.0475 0 0" rpy="0 0 0"/>
-  </xacro:dispensing>
   <link name="conveyor">
     <visual>

File: src/tools_manager/urdf/tool_mount.urdf.xacro (robot description, xacro)
@@ -6,14 +6,10 @@
     mount_origin_xyz:='0 0 0'
     mount_origin_rpy:='0 0 0'
-    tcp_origin_xyz:='0 0 0'
-    tcp_origin_rpy:='0 0 0'
     ">
-    <link name="tool_mount_link">
+    <link name="tool_mount_tcp">
         <visual>
             <origin xyz="0 0 0" rpy="0 0 0"/>
             <geometry>
-                <mesh>
-                <uri>model://tool_mount/meshes/visual.dae</uri>
-                </mesh>
+                <mesh filename="model://tool_mount/meshes/visual.dae"/>
             </geometry>
         </visual>
@@ -21,32 +17,31 @@
             <origin xyz="0 0 0" rpy="0 0 0"/>
             <geometry>
-                <mesh>
-                <uri>model://tool_mount/meshes/collision.stl</uri>
-                </mesh>
+                <mesh filename="model://tool_mount/meshes/collision.stl"/>
             </geometry>
         </collision>
         <inertial>
-            <mass value="0.5"/>
-            <inertia ixx="0.001" ixy="0" ixz="0" iyy="0.001" iyz="0" izz="0.001"/>
+            <origin xyz="0 0 0" rpy="0 0 0"/>
+            <mass value="4.697067588322115"/>
+            <inertia
+                ixx="1.841474459710298"
+                ixy="-0.004289082833111024"
+                ixz="0.10558599010118996"
+                iyy="1.824344061067677"
+                iyz="0.029655588824880397"
+                izz="2.055971309702727"/>
         </inertial>
     </link>
-    <disable_collisions link1="tool_mount_link" link2="${parent}" reason="Adjacent" />
-    <joint name="tool_mount_joint" type="fixed">
+    <disable_collisions link1="tool_mount_tcp" link2="${parent}" reason="Adjacent" />
+    <joint name="tool_mount_tcp_joint" type="fixed">
         <parent link="${parent}"/>
-        <child link="tool_mount_link"/>
+        <child link="tool_mount_tcp"/>
         <origin xyz="${mount_origin_xyz}" rpy="${mount_origin_rpy}"/>
-    </joint>
-    <link name="tool_mount_tcp"/>
-    <joint name="tool_mount_to_tool_tcp_joint" type="fixed">
-        <parent link="tool_mount_link"/>
-        <child link="tool_mount_tcp"/>
-        <origin xyz="${tcp_origin_xyz}" rpy="${tcp_origin_rpy}"/>
     </joint>
     <xacro:if value="${simulated}">
         <link name="rfid_scanner_link"/>
         <joint name="tool_mount_to_rfid_scanner_joint" type="fixed">
-            <parent link="tool_mount_link"/>
+            <parent link="tool_mount_tcp"/>
             <child link="rfid_scanner_link"/>
-            <origin xyz="0 0 0" rpy="0 0 0"/>
+            <origin xyz="0.0778 0 -0.033" rpy="0 0 0"/>
         </joint>
         <gazebo>
@@ -54,5 +49,5 @@
                     name="autofactory::rfid::RfidReader">
                 <link>rfid_scanner_link</link>
-                <range>0.1</range>
+                <range>0.02</range>
                 <update_rate>10</update_rate>
                 <detected_topic>/tool_mount_rfid_scanner/detected</detected_topic>

File: src/tools_manager/urdf/tool_rack.urdf.xacro (robot description, xacro)
@@ -10,11 +10,13 @@
     index:='2'
     parent:='tool_rack_link'
-    x_offset:='0'
-    tool_attached_origin_xyz:='0.1 0 0'
+    y_offset:='0'
+    tool_attached_origin_xyz:='0.0256 -0.1025 0.287'
     tool_attached_origin_rpy:='0 0 0'
-    tool_lifted_origin_xyz:='0.1 0 0'
+    tool_lifted_origin_xyz:='0.0256 -0.1025 0.4'
     tool_lifted_origin_rpy:='0 0 0'
-    tool_slide_in_origin_xyz:='0.1 0 0'
+    tool_slide_in_origin_xyz:='0.0656 -0.1025 0.287'
     tool_slide_in_origin_rpy:='0 0 0'
+    rfid_scanner_origin_xyz:='-0.02 -0.1025 0.23'
+    rfid_scanner_origin_rpy:='0 0 0'
     ">
     <link name="slot${index}_attached_link"/>
@@ -22,5 +24,5 @@
         <parent link="${parent}"/>
         <child link="slot${index}_attached_link"/>
-        <origin xyz="${float(tool_attached_origin_xyz.split()[0]) + float(x_offset)} ${tool_attached_origin_xyz.split()[1]} ${tool_attached_origin_xyz.split()[2]}" rpy="${tool_attached_origin_rpy}"/>
+        <origin xyz="${tool_attached_origin_xyz.split()[0]} ${float(tool_attached_origin_xyz.split()[1]) + float(y_offset)} ${tool_attached_origin_xyz.split()[2]}" rpy="${tool_attached_origin_rpy}"/>
     </joint>
     <link name="slot${index}_lifted_link"/>
@@ -28,5 +30,5 @@
         <parent link="${parent}"/>
         <child link="slot${index}_lifted_link"/>
-        <origin xyz="${float(tool_lifted_origin_xyz.split()[0]) + float(x_offset)} ${tool_lifted_origin_xyz.split()[1]} ${tool_lifted_origin_xyz.split()[2]}" rpy="${tool_lifted_origin_rpy}"/>
+        <origin xyz="${tool_lifted_origin_xyz.split()[0]} ${float(tool_lifted_origin_xyz.split()[1]) + float(y_offset)} ${tool_lifted_origin_xyz.split()[2]}" rpy="${tool_lifted_origin_rpy}"/>
     </joint>
     <link name="slot${index}_slide_in_link"/>
@@ -34,5 +36,5 @@
         <parent link="${parent}"/>
         <child link="slot${index}_slide_in_link"/>
-        <origin xyz="${float(tool_slide_in_origin_xyz.split()[0]) + float(x_offset)} ${tool_slide_in_origin_xyz.split()[1]} ${tool_slide_in_origin_xyz.split()[2]}" rpy="${tool_slide_in_origin_rpy}"/>
+        <origin xyz="${tool_slide_in_origin_xyz.split()[0]} ${float(tool_slide_in_origin_xyz.split()[1]) + float(y_offset)} ${tool_slide_in_origin_xyz.split()[2]}" rpy="${tool_slide_in_origin_rpy}"/>
     </joint>
     <xacro:if value="${simulated}">
@@ -41,5 +43,5 @@
             <parent link="slot${index}_attached_link"/>
             <child link="slot${index}_rfid_scanner_link"/>
-            <origin xyz="0 0 0" rpy="0 0 0"/>
+            <origin xyz="${rfid_scanner_origin_xyz.split()[0]} ${float(rfid_scanner_origin_xyz.split()[1]) + float(y_offset)} ${rfid_scanner_origin_xyz.split()[2]}" rpy="${rfid_scanner_origin_rpy}"/>
         </joint>
         <gazebo>
@@ -67,5 +69,5 @@
             index="${index}"
             parent="${parent}"
-            x_offset="${index * spacing}"/>
+            y_offset="${index * spacing}"/>
         <xacro:tool_slots
             simulated="${simulated}"
@@ -89,7 +91,5 @@
             <origin xyz="0 0 0" rpy="0 0 0"/>
             <geometry>
-                <mesh>
-                <uri>model://tool_rack/meshes/visual.dae</uri>
-                </mesh>
+                <mesh filename="model://tool_rack/meshes/visual.dae"/>
             </geometry>
         </visual>
@@ -97,7 +97,5 @@
             <origin xyz="0 0 0" rpy="0 0 0"/>
             <geometry>
-                <mesh>
-                <uri>model://tool_rack/meshes/collision.stl</uri>
-                </mesh>
+                <mesh filename="model://tool_rack/meshes/collision.stl"/>
             </geometry>
         </collision>

Commit message: move the tool_rack to correct place; add material color

File: src/cameras/urdf/basler.urdf.xacro (robot description, xacro)
@@ -40,4 +40,7 @@
           </xacro:unless>
         </geometry>
+        <material name="tool_rack_grey">
+            <color rgba="0.5 0.5 0.5 1"/>
+        </material>
       </visual>
       <collision>

File: src/laser_sensors/urdf/cross_laser.urdf.xacro (robot description, xacro)
@@ -17,4 +17,7 @@
             <mesh filename="file://${laser_sensors_model_base}/captron/meshes/sensor_visual.dae"/>
         </geometry>
+        <material name="tool_rack_grey">
+            <color rgba="0.5 0.5 0.5 1"/>
+        </material>
       </visual>
       <collision>

File: src/station/config/urdf/ur/gz_sim.urdf.xacro (robot description, xacro)
@@ -77,4 +77,7 @@
         <mesh filename="file://$(find station)/config/model/station/meshes/station_visual.dae"/>
       </geometry>
+      <material name="tool_rack_grey">
+          <color rgba="0.5 0.5 0.5 1"/>
+      </material>
     </visual>
     <collision>
@@ -99,5 +102,5 @@
     parent="station"
     simulated="true"
-    rack_origin_xyz="0.3 -0.7 0.9"
+    rack_origin_xyz="-0.03 -0.427 0.9"
     rack_origin_rpy="0 0 1.5708"
     number_of_slots="2"

File: src/station/config/urdf/ur/real.urdf.xacro (robot description, xacro)
@@ -90,4 +90,7 @@
         <mesh filename="file://$(find station)/config/model/station/meshes/station_visual.dae"/>
       </geometry>
+      <material name="tool_rack_grey">
+          <color rgba="0.5 0.5 0.5 1"/>
+      </material>
     </visual>
     <collision>
@@ -112,5 +115,5 @@
     parent="station"
     simulated="false"
-    rack_origin_xyz="0.35 -0.4 0.9"
+    rack_origin_xyz="-0.03 -0.427 0.9"
     rack_origin_rpy="0 0 0"
     number_of_slots="2"

File: src/tools_manager/urdf/tool_mount.urdf.xacro (robot description, xacro)
@@ -18,4 +18,7 @@
                 <mesh filename="file://$(find tools_manager)/model/tool_mount/meshes/visual.dae"/>
             </geometry>
+            <material name="tool_mount_grey">
+                <color rgba="0.5 0.5 0.5 1"/>
+            </material>
         </visual>
         <collision>

File: src/tools_manager/urdf/tool_rack.urdf.xacro (robot description, xacro)
@@ -129,4 +129,7 @@
                 <mesh filename="file://$(find tools_manager)/model/tool_rack/meshes/visual.dae"/>
             </geometry>
+            <material name="tool_rack_grey">
+                <color rgba="0.5 0.5 0.5 1"/>
+            </material>
         </visual>
         <collision>

Commit message: correct camera view in simulation

File: src/cameras/urdf/basler.urdf.xacro (robot description, xacro)
@@ -89,5 +89,5 @@
         <child link="camera_tcp_uncalibrated"/>
         <xacro:if value="${camera_model == 'basler'}">
-            <origin xyz="0.0188 0.0395 -0.0695" rpy="0 0 0"/>
+            <origin xyz="0.0188 0.0395 -0.0695" rpy="0 1.5707963267948966 0"/>
         </xacro:if>
         <xacro:unless value="${is_known_model}">
