Commit message: update cross-laser links and example script

File: src/laser_sensors/urdf/cross_laser.urdf.xacro (robot description, xacro)
@@ -42,5 +42,5 @@
       <parent link="${name}_laser_sensor_link"/>
       <child link="${name}_orl2_intersection"/>
-      <origin xyz="0 -0.0425 0.02591" rpy="0 0 0"/>
+      <origin xyz="0 -0.0425 0.02591" rpy="0 0 -3.141592653589793"/>
     </joint>
     <!--
